Commit message: refactor: xacro inertia added to URDF

File: src/my_trirob_description/urdf/my_trirob.urdf.xacro (robot description, xacro)
@@ -20,4 +20,6 @@
     <xacro:example_macro a="2" b="3" c="4" />
 -->
+<!--I will include the common properties file here-->
+    <xacro:include filename="common_properties.xacro" />
     <xacro:macro name="wheel_link" params="prefix" >
         <link name="${prefix}_wheel_link" >
@@ -29,4 +31,6 @@
                 <material name="grey" />
             </visual>
+            <xacro:cylinder_inertia m="1.0" r="${wheel_radius}" h="${wheel_length}"
+                                   xyz="0 0 0" rpy="${pi / 2.0} 0 0" />
         </link>
     </xacro:macro>
@@ -45,7 +49,9 @@
                 <box size="${base_length} ${base_width} ${base_height}"/>
             </geometry>
-            <origin xyz="0 0 0.1" rpy="0 0 0"/>
+            <origin xyz="0 0 ${base_height / 2.0}" rpy="0 0 0"/>
             <material name="green"/>
         </visual>
+        <xacro:box_inertia m="5.0" l="${base_length}" w="${base_width}" h="${base_height}"
+                           xyz="0  0 ${base_height / 2.0}" rpy="0 0 0" />
     </link>
 <!--
@@ -77,4 +83,6 @@
             <material name="grey" />
         </visual>
+        <xacro:sphere_inertia m="0.5" r="${wheel_radius / 2.0}"
+                              xyz="0 0 0" rpy="0 0 0" />
     </link>
     <!--TF-->

Commit message: feat: collision enabled

File: src/my_trirob_description/urdf/my_trirob.urdf.xacro (robot description, xacro)
@@ -31,4 +31,10 @@
                 <material name="grey" />
             </visual>
+            <collision>
+                <geometry>
+                    <cylinder radius="${wheel_radius}" length="${wheel_length}" />
+                </geometry>
+                <origin xyz="0 0 0" rpy="${pi / 2.0} 0 0" />
+            </collision>
             <xacro:cylinder_inertia m="1.0" r="${wheel_radius}" h="${wheel_length}"
                                    xyz="0 0 0" rpy="${pi / 2.0} 0 0" />
@@ -52,4 +58,10 @@
             <material name="green"/>
         </visual>
+        <collision>
+            <geometry>
+                <box size="${base_length} ${base_width} ${base_height}"/>
+            </geometry>
+            <origin xyz="0 0 ${base_height / 2.0}" rpy="0 0 0"/>
+        </collision>
         <xacro:box_inertia m="5.0" l="${base_length}" w="${base_width}" h="${base_height}"
                            xyz="0  0 ${base_height / 2.0}" rpy="0 0 0" />
@@ -83,4 +95,10 @@
             <material name="grey" />
         </visual>
+        <collision>
+            <geometry>
+                <sphere radius="${wheel_radius / 2.0}" />
+            </geometry>
+            <origin xyz="0 0 0" rpy="0 0 0"/>
+        </collision>
         <xacro:sphere_inertia m="0.5" r="${wheel_radius / 2.0}"
                               xyz="0 0 0" rpy="0 0 0" />
